Commit message: Update brain_turtlebot's model

File: turtlebot3/turtlebot3_description/urdf/turtlebot3_waffle_pi.gazebo.xacro (robot description, xacro)
@@ -5,5 +5,5 @@
   <xacro:arg name="imu_visual"    default="false"/>
   <gazebo reference="base_link">
-    <material>Gazebo/DarkGrey</material>
+    <material>Gazebo/Yellow</material>
   </gazebo>
   <gazebo reference="wheel_left_link">
@@ -135,34 +135,5 @@
   </gazebo>
   <gazebo reference="high_scan">
-    <material>Gazebo/FlatBlack</material>
-    <sensor type="ray" name="lds_lfcd_sensor_2">
-      <pose>0 0 0 0 0 0</pose>
-      <visualize>false</visualize>
-      <update_rate>200</update_rate>
-      <ray>
-        <scan>
-          <horizontal>
-            <samples>360</samples>
-            <resolution>1</resolution>
-            <min_angle>0.0</min_angle>
-            <max_angle>6.28319</max_angle>
-          </horizontal>
-        </scan>
-        <range>
-          <min>0.120</min>
-          <max>3.5</max>
-          <resolution>0.015</resolution>
-        </range>
-        <!-- <noise>
-          <type>gaussian</type>
-          <mean>0.0</mean>
-          <stddev>0.01</stddev>
-        </noise> -->
-      </ray>
-      <plugin name="gazebo_ros_lds_lfcd_controller_2" filename="libgazebo_ros_laser.so">
-        <topicName>scanhigh</topicName>
-        <frameName>high_scan</frameName>
-      </plugin>
-    </sensor>
+    <material>Gazebo/Red</material>
   </gazebo>
 <!--link : https://www.raspberrypi.org/documentation/hardware/camera/-->

File: turtlebot3/turtlebot3_description/urdf/turtlebot3_waffle_pi.urdf.xacro (robot description, xacro)
@@ -188,5 +188,5 @@
     <parent link="base_scan"/>
     <child link="high_scan"/>
-    <origin xyz="0 0 0.15" rpy="0 0 0"/>
+    <origin xyz="0.2 0 0" rpy="0 0 0"/>
   </joint>
   <link name="high_scan">
